Commit message: It pybullet param all setting done

File: src/robot_description/urdf/target.urdf (robot description, URDF)
Before this commit: robot angle_excurate_arm_ver2, 9 links, 8 joints
Links:
- removed link base_link2_v2_1
- removed link base_link_2_1
- removed link camera_1
- removed link link3_v1_1
- removed link link4_v1_1
- removed link robot_ver7_grap1_2_v1_1
- removed link robot_ver7_grap2_2_v1_1
- removed link robot_ver7_link_4_v1_1
- added link 14joint44v2_1, mass 6.462489586316137; collision mesh filename=package://robot_description/meshes/14joint44v2_1.stl scale=0.001 0.001 0.001; visual mesh filename=package://robot_description/meshes/14joint44v2_1.stl scale=0.001 0.001 0.001
- added link 25joint_v2_1, mass 15.540708623156803; collision mesh filename=package://robot_description/meshes/25joint_v2_1.stl scale=0.001 0.001 0.001; visual mesh filename=package://robot_description/meshes/25joint_v2_1.stl scale=0.001 0.001 0.001
- added link 25jointt_1, mass 15.540708623156789; collision mesh filename=package://robot_description/meshes/25jointt_1.stl scale=0.001 0.001 0.001; visual mesh filename=package://robot_description/meshes/25jointt_1.stl scale=0.001 0.001 0.001
- added link board_1, mass 0.3723965227028356; collision mesh filename=package://robot_description/meshes/board_1.stl scale=0.001 0.001 0.001; visual mesh filename=package://robot_description/meshes/board_1.stl scale=0.001 0.001 0.001
- added link cralwer_deap2_1, mass 0.2861324999999951; collision mesh filename=package://robot_description/meshes/cralwer_deap2_1.stl scale=0.001 0.001 0.001; visual mesh filename=package://robot_description/meshes/cralwer_deap2_1.stl scale=0.001 0.001 0.001
- added link cralwer_deap_1, mass 0.28613249999999474; collision mesh filename=package://robot_description/meshes/cralwer_deap_1.stl scale=0.001 0.001 0.001; visual mesh filename=package://robot_description/meshes/cralwer_deap_1.stl scale=0.001 0.001 0.001
- added link craw_1, mass 2.052982330856382; collision mesh filename=package://robot_description/meshes/craw_1.stl scale=0.001 0.001 0.001; visual mesh filename=package://robot_description/meshes/craw_1.stl scale=0.001 0.001 0.001
- added link flange_1, mass 1.2487889322710095; collision mesh filename=package://robot_description/meshes/flange_1.stl scale=0.001 0.001 0.001; visual mesh filename=package://robot_description/meshes/flange_1.stl scale=0.001 0.001 0.001
- added link joint143_1, mass 6.462489586316132; collision mesh filename=package://robot_description/meshes/joint143_1.stl scale=0.001 0.001 0.001; visual mesh filename=package://robot_description/meshes/joint143_1.stl scale=0.001 0.001 0.001
- added link joint14_1, mass 6.462489586316139; collision mesh filename=package://robot_description/meshes/joint14_1.stl scale=0.001 0.001 0.001; visual mesh filename=package://robot_description/meshes/joint14_1.stl scale=0.001 0.001 0.001
- added link joint252_1, mass 15.540708623156794; collision mesh filename=package://robot_description/meshes/joint252_1.stl scale=0.001 0.001 0.001; visual mesh filename=package://robot_description/meshes/joint252_1.stl scale=0.001 0.001 0.001
- added link larm_1, mass 0.0; collision mesh filename=package://robot_description/meshes/larm_1.stl scale=0.001 0.001 0.001; visual mesh filename=package://robot_description/meshes/larm_1.stl scale=0.001 0.001 0.001
- added link transv2_1, mass 9.761584230310485; collision mesh filename=package://robot_description/meshes/transv2_1.stl scale=0.001 0.001 0.001; visual mesh filename=package://robot_description/meshes/transv2_1.stl scale=0.001 0.001 0.001
- added link uarm_1, mass 0.0; collision mesh filename=package://robot_description/meshes/uarm_1.stl scale=0.001 0.001 0.001; visual mesh filename=package://robot_description/meshes/uarm_1.stl scale=0.001 0.001 0.001
- added link virtual_tip_link, mass 0.00001
- link base_link: mass 7.925585093654501e-07 -> 7.803232490794544
Joints:
- removed joint Revolute 1
- removed joint Revolute 2
- removed joint Revolute 3
- removed joint Revolute 4
- removed joint Revolute 5
- removed joint Revolute 6
- removed joint Rigid 11
- removed joint Rigid 8
- added joint Revolute 21: type continuous, parent base_link, child joint252_1, origin xyz=0.001849 0.003782 0.07 rpy=0 0 0, axis 0.0 0.0 1.0
- added joint Revolute 34: type continuous, parent 25jointt_1, child transv2_1, origin xyz=0.0 0.071 0.066501 rpy=0 0 0, axis 0.0 -1.0 0.0
- added joint Revolute 40: type continuous, parent joint14_1, child 14joint44v2_1, origin xyz=0.0 -0.058 0.049 rpy=0 0 0, axis 0.0 -1.0 -0.0
- added joint Revolute 41: type continuous, parent 14joint44v2_1, child joint143_1, origin xyz=0.0 -0.049 0.058 rpy=0 0 0, axis 0.0 -0.0 1.0
- added joint Revolute 42: type continuous, parent joint143_1, child flange_1, origin xyz=0.0 -0.058 0.049 rpy=0 0 0, axis 0.0 -1.0 -0.0
- added joint Revolute_22: type revolute, parent joint252_1, child 25joint_v2_1, origin xyz=0.0 -0.069999 0.076501 rpy=0 0 0, axis 0.0 -1.0 0.0, limit lower=-1.47 upper=1.47 effort=10 velocity=1.0
- added joint Rigid 30: type fixed, parent 25joint_v2_1, child larm_1, origin xyz=0.0 -0.071 0.066501 rpy=0 0 0
- added joint Rigid 32: type fixed, parent larm_1, child 25jointt_1, origin xyz=0.0 0.0 0.268085 rpy=0 0 0
- added joint Rigid 35: type fixed, parent transv2_1, child uarm_1, origin xyz=0.0 0.045 0.0651 rpy=0 0 0
- added joint Rigid 37: type fixed, parent uarm_1, child joint14_1, origin xyz=0.0 0.0 0.227 rpy=0 0 0
- added joint Rigid 43: type fixed, parent flange_1, child board_1, origin xyz=0.0 -0.0315 0.0 rpy=0 0 0
- added joint Rigid 44: type fixed, parent board_1, child craw_1, origin xyz=-0.0345 -0.006 0.0595 rpy=0 0 0
- added joint Slider 52: type prismatic, parent craw_1, child cralwer_deap_1, origin xyz=0.009 -0.054 -0.00325 rpy=0 0 0, axis 1.0 -0.0 -0.0, limit lower=-0.01 upper=0.01 effort=100 velocity=100
- added joint Slider 53: type prismatic, parent craw_1, child cralwer_deap2_1, origin xyz=0.063 -0.054 -0.00325 rpy=0 0 0, axis 1.0 -0.0 -0.0, limit lower=-0.01 upper=0.01 effort=100 velocity=100
- added joint virtual_tip_joint: type revolute, parent craw_1, child virtual_tip_link, origin xyz= 0.036 -0.054 -0.00325 rpy=0 0 0, axis 0 0 1, limit lower=0 upper=0 effort=0 velocity=0

Commit message: up down left right can use

File: src/robot_description/urdf/target.urdf (robot description, URDF)
Before this commit: robot with_craw, 16 links, 15 joints
Joints:
- joint virtual_tip_joint: axis 0 0 1 -> 1 0 0; origin xyz= 0.036 -0.054 -0.00325 rpy=0 0 0 -> xyz= 0.036 -0.054 -0.00325 rpy=3.14 3.14 1.57
